File: OBC/OBC_KICAD/JST_Debugger.kicad_sch (KiCad schematic)
At the start: 5 parts, among them J5 USB_C_Receptacle_USB2.0_14P, J6 Screw_Terminal_01x05, U5 USBLC6-2SC6

Commit message: Update
Parts:
- added J1: Screw_Terminal_01x02, symbol Connector:Screw_Terminal_01x02
Other:
- note added: "UART COM"
Changed lines of the file:
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@@
+		)
+	)
+	(text "UART COM\n"
+		(exclude_from_sim no)
+		(at 100.838 36.322 0)
+		(effects
+			(font
+				(size 1.27 1.27)
+			)
 		)
 	)
@@
 					(unit 1)
 				)
+			)
+		)
+	)
+	(symbol
+		(lib_id "Connector:Screw_Terminal_01x02")
+		(at 96.52 43.18 0)
+		(unit 1)
+		(exclude_from_sim no)
+		(in_bom yes)
+		(on_board yes)
+		(dnp no)
+		(fields_autoplaced yes)
+		(property "Reference" "J1"
+			(at 99.06 43.1799 0)
+			(effects
+				(font
+					(size 1.27 1.27)
+				)
+				(justify left)
+			)
+		)
+		(property "Value" "Screw_Terminal_01x02"
+			(at 99.06 45.7199 0)
+			(effects
+				(font
+					(size 1.27 1.27)
+				)
+				(justify left)
+			)
+		)
+		(property "Footprint" ""
+			(at 96.52 43.18 0)
+			(effects
+				(font
+					(size 1.27 1.27)
+				)
+				(hide yes)
+			)
+		)
+		(property "Datasheet" "~"
+			(at 96.52 43.18 0)
+			(effects
+				(font
+					(size 1.27 1.27)
+				)
+				(hide yes)
+			)
+		)
+		(property "Description" "Generic screw terminal, single row, 01x02, script generated (kicad-library-utils/schlib/autogen/connector/)"
+			(at 96.52 43.18 0)
+			(effects
+				(font
+					(size 1.27 1.27)
+				)
+				(hide yes)
+			)
+		)
+		(pin "1"
+		)
+		(pin "2"
+		)
+		(instances
+			(project ""
+				(path "/6db8dc25-5ab8-4f32-8d05-e8d57edb0b6f/709184b9-2641-4adb-9bb3-7646cf8c1857"
+					(reference "J1")
+					(unit 1)
+				)

Commit message: Cirtcuito Completo
Circuito Completo
Parts:
- removed J1: Screw_Terminal_01x02, symbol Connector:Screw_Terminal_01x02
- removed J6: Screw_Terminal_01x05, symbol Connector:Screw_Terminal_01x05
- added C23: 100n, Capacitor_SMD:C_0805_2012Metric_Pad1.18x1.45mm_HandSolder, symbol Device:C
- added D1: 1N4148W, Diode_SMD:D_SOD-123, symbol Diode:1N4148W
- added J1: Conn_01x05, Connector_PinSocket_2.54mm:PinSocket_1x05_P2.54mm_Vertical_SMD_Pin1Left, symbol Connector_Generic:Conn_01x05
- added U6: AMS1117-3.3, Package_TO_SOT_SMD:SOT-223-3_TabPin2, symbol Regulator_Linear:AMS1117-3.3
- J5: footprint (none) -> Connector_USB:USB_C_Receptacle_GCT_USB4110
- R15, R16: footprint (none) -> Resistor_SMD:R_0805_2012Metric_Pad1.20x1.40mm_HandSolder
Connections:
- net GND: now also C23.2, J1.5 (Pin_5), U6.1 (GND)
- net SWCLK: now also J1.2 (Pin_2)
- net SWDIO: now also J1.3 (Pin_3)
- net at J5.A4 (VBUS), J5.A9 (VBUS), J5.B4 (VBUS)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: now also U6.3 (VI)
- new net: C23.1, D1.2 (A), U6.2 (VO)
- new net NRST_PROGRAM: J1.4 (Pin_4)
- new net VCC_OBC: D1.1 (K), J1.1 (Pin_1)
Other:
- note removed: "UART COM"
- title: (none) -> David_Moises_Garcia_Sopino_Hoja2_IIS
