File: OBC/OBC_KICAD/OBC_KICAD.kicad_pcb (KiCad board)
At the start: 2 copper layers, 7 parts, among them J3 Conn_01x02, J4 Conn_01x02, U1 STWD100YNYWY3F, U2 STM32F405RGTx, U3 TPS2052BDR, U5 USBLC6-2SC6

Commit message: Cirtcuito Completo
Circuito Completo
Parts:
- removed J3, J4: Conn_01x02, Connector_JST:JST_PH_B2B-PH-K_1x02_P2.00mm_Vertical
- removed U3: TPS2052BDR, TPS2052BDR:SOIC127P599X175-8N
- added C10: 2.2uF, Capacitor_SMD:C_0805_2012Metric_Pad1.18x1.45mm_HandSolder, F.Cu at (155.2, 85.8)
- added C12: 100n, Capacitor_SMD:C_0805_2012Metric_Pad1.18x1.45mm_HandSolder, F.Cu at (135.7, 96.4)
- added C14: 1u, Capacitor_SMD:C_0805_2012Metric_Pad1.18x1.45mm_HandSolder, F.Cu at (131.8, 96.4)
- added C15: 10u, Capacitor_SMD:C_0805_2012Metric_Pad1.18x1.45mm_HandSolder, F.Cu at (161.7, 113.7)
- added C16: 100n, Capacitor_SMD:C_0805_2012Metric_Pad1.18x1.45mm_HandSolder, F.Cu at (167.5, 113.6)
- added C17: 0.1u, Capacitor_SMD:C_0805_2012Metric_Pad1.18x1.45mm_HandSolder, F.Cu at (167.6, 71.5)
- added C18: 4.7u, Capacitor_SMD:C_0805_2012Metric_Pad1.18x1.45mm_HandSolder, F.Cu at (116.7, 84.2)
- added C19: 4.7u, Capacitor_SMD:C_0805_2012Metric_Pad1.18x1.45mm_HandSolder, F.Cu at (152.7, 69.2)
- added C2: 100n, Capacitor_SMD:C_0805_2012Metric_Pad1.18x1.45mm_HandSolder, F.Cu at (121.9, 84.3)
- added C20: 22u, Capacitor_SMD:C_0805_2012Metric_Pad1.18x1.45mm_HandSolder, F.Cu at (161.2, 68.8)
- added C21: 15pF, Capacitor_SMD:C_0805_2012Metric_Pad1.18x1.45mm_HandSolder, F.Cu at (122.6, 91.7)
- added C22: 15pF, Capacitor_SMD:C_0805_2012Metric_Pad1.18x1.45mm_HandSolder, F.Cu at (126.3, 91.7)
- added C23: 100n, Capacitor_SMD:C_0805_2012Metric_Pad1.18x1.45mm_HandSolder, F.Cu at (118.0, 78.2)
- added C3: 10u, Capacitor_SMD:C_0805_2012Metric_Pad1.18x1.45mm_HandSolder, F.Cu at (128.2, 96.4)
- added C4: 100n, Capacitor_SMD:C_0805_2012Metric_Pad1.18x1.45mm_HandSolder, F.Cu at (126.4, 84.2)
- added C5: 100n, Capacitor_SMD:C_0805_2012Metric_Pad1.18x1.45mm_HandSolder, F.Cu at (124.7, 96.4)
- added C6: 100n, Capacitor_SMD:C_0805_2012Metric_Pad1.18x1.45mm_HandSolder, F.Cu at (130.4, 84.2)
- added C7: 100n, Capacitor_SMD:C_0805_2012Metric_Pad1.18x1.45mm_HandSolder, F.Cu at (134.4, 84.2)
- added C8: 2.2 uF, Capacitor_SMD:C_0805_2012Metric_Pad1.18x1.45mm_HandSolder, F.Cu at (146.2, 101.7)
- added C9: 100n, Capacitor_SMD:C_0805_2012Metric_Pad1.18x1.45mm_HandSolder, F.Cu at (137.9, 84.2)
- added CARD1: MICRO SD, Connector_Card:microSD_HC_Hirose_DM3AT-SF-PEJM5, F.Cu at (169.9, 100.3)
- added D1: 1N4148W, Diode_SMD:D_SOD-123, F.Cu at (124.2, 78.2)
- added D2: 1N4148W, Diode_SMD:D_SOD-123, F.Cu at (167.3, 65.0)
- added FB1: FerriteBead, Inductor_SMD:L_Walsin_WLFM252009x, F.Cu at (120.5, 96.7)
- added H1: MountingHole, MountingHole:MountingHole_3.2mm_M3_Pad_Via, F.Cu at (180.1, 132.5)
- added H2: MountingHole, MountingHole:MountingHole_3.2mm_M3_Pad_Via, F.Cu at (180.1, 52.5)
- added H3: MountingHole, MountingHole:MountingHole_3.2mm_M3_Pad_Via, F.Cu at (100.1, 132.5)
- added H4: MountingHole, MountingHole:MountingHole_3.2mm_M3_Pad_Via, F.Cu at (100.1, 52.5)
- added J1: Conn_01x05, Connector_PinSocket_2.54mm:PinSocket_1x05_P2.54mm_Vertical_SMD_Pin1Left, F.Cu at (121.9, 122.7)
- added J2: Conn_02x20_Counter_Clockwise, Connector_PinSocket_2.54mm:PinSocket_2x20_P2.54mm_Vertical, F.Cu at (116.0, 53.1)
- added J5: USB_C_Receptacle_USB2.0_14P, Connector_USB:USB_C_Receptacle_GCT_USB4110, F.Cu at (109.2, 69.7)
- added R1: 10k, Resistor_SMD:R_0805_2012Metric_Pad1.20x1.40mm_HandSolder, F.Cu at (143.8, 80.7)
- added R12: 10k, Resistor_SMD:R_0805_2012Metric_Pad1.20x1.40mm_HandSolder, F.Cu at (167.6, 61.7)
- added R15: 5k1, Resistor_SMD:R_0805_2012Metric_Pad1.20x1.40mm_HandSolder, F.Cu at (117.5, 63.0)
- added R16: 5k1, Resistor_SMD:R_0805_2012Metric_Pad1.20x1.40mm_HandSolder, F.Cu at (105.2, 80.8)
- added R2: 47K, Resistor_SMD:R_0805_2012Metric_Pad1.20x1.40mm_HandSolder, F.Cu at (146.2, 74.0)
- added R3: 47K, Resistor_SMD:R_0805_2012Metric_Pad1.20x1.40mm_HandSolder, F.Cu at (150.1, 74.0)
- added R4: 47K, Resistor_SMD:R_0805_2012Metric_Pad1.20x1.40mm_HandSolder, F.Cu at (154.7, 74.0)
- added R5: 47K, Resistor_SMD:R_0805_2012Metric_Pad1.20x1.40mm_HandSolder, F.Cu at (158.8, 74.0)
- added R6: 47K, Resistor_SMD:R_0805_2012Metric_Pad1.20x1.40mm_HandSolder, F.Cu at (162.7, 74.0)
- added R7: 100k, Resistor_SMD:R_0805_2012Metric_Pad1.20x1.40mm_HandSolder, F.Cu at (155.5, 110.6)
- added R8: 4.7k, Resistor_SMD:R_0805_2012Metric_Pad1.20x1.40mm_HandSolder, F.Cu at (164.9, 81.8)
- added SwReset1: SW_Push, Button_Switch_SMD:SW_Push_1P1T_NO_CK_PTS125Sx43PSMTR, F.Cu at (177.4, 71.3)
- added U4: TPS2052BDR, TPS2052BDR:SOIC127P599X175-8N, F.Cu at (159.5, 63.5)
- added U6: AMS1117-3.3, Package_TO_SOT_SMD:SOT-223-3_TabPin2, F.Cu at (124.2, 71.6)
- added XTAL1: ECS-80-12-30BQ-JES-TR, esc_cristal:ECS-80-12_ECS, F.Cu at (132.5, 89.2)
- moved U2 29.1 mm to (145.0, 92.0)
- moved U1 24.8 mm to (167.5, 86.5)
- moved U5 24.4 mm to (110.2, 84.3)
- moved SwBoot1 21.8 mm to (177.7, 87.0)
Connections:
- net +3V3 renamed VCC_OBC
- U2 pad 10: MISO_BM -> CardDetect
- U2 pad 11: MOSI_BM -> unconnected-(U2-PC3-Pad11)
- U2 pad 13: +3.3VA -> +3V3A
- U2 pad 14: ELRS_UART_TX -> TX
- U2 pad 15: ELRS_UART_RX -> RX
- U2 pad 16: unconnected-(U2-PA2-Pad16) -> IEPS
- U2 pad 20: AP_CS_IMU -> CS
- U2 pad 21: CLK_IMU -> SCK
- U2 pad 22: MISO_IMU -> MISO
- U2 pad 23: MOSI_IMU -> MOSI
- U2 pad 26: CS_BM -> unconnected-(U2-PB0-Pad26)
- U2 pad 29: SCK_BM -> En_P1
- U2 pad 3: /Microcontrolador/LSE_IN -> unconnected-(U2-PC14-Pad3)
- U2 pad 30: unconnected-(U2-PB11-Pad30) -> En_P2
- U2 pad 33: unconnected-(U2-PB12-Pad33) -> En_ADC
- U2 pad 34: unconnected-(U2-PB13-Pad34) -> En_COM
- U2 pad 4: /Microcontrolador/LSE_OUT -> unconnected-(U2-PC15-Pad4)
- U2 pad 42: TX_VTX -> unconnected-(U2-PA9-Pad42)
- U2 pad 43: RX_VTX -> unconnected-(U2-PA10-Pad43)
- U2 pad 58: SCL_MAG -> SCL
- U2 pad 59: SDA_MAG -> SDA
- U2 pad 8: EN1P1 -> NRST_PROGRAM
- U2 pad 9: EN2P2 -> unconnected-(U2-PC1-Pad9)
Routing:
- net GND: track 0.00 -> 154.8 mm, vias 0 -> 38
- net VCC_OBC: track 0.00 -> 102.2 mm, vias 0 -> 20
- net En_P2: track 0.00 -> 87.7 mm, vias 0 -> 2
- net En_P1: track 0.00 -> 84.6 mm, vias 0 -> 2
- net /Microcontrolador/RESET: track 0.00 -> 78.0 mm, vias 0 -> 4
- net IEPS: track 0.00 -> 77.8 mm, vias 0 -> 2
- net En_ADC: track 0.00 -> 58.8 mm, vias 0 -> 2
- net SWCLK: track 0.00 -> 57.1 mm, vias 0 -> 2
- net SWDIO: track 0.00 -> 56.8 mm
- net MOSI: track 0.00 -> 55.8 mm, vias 0 -> 3
- net +3V3: track 0.00 -> 52.2 mm, vias 0 -> 1
- net NRST_PROGRAM: track 0.00 -> 52.0 mm, vias 0 -> 2
- net CS: track 0.00 -> 51.0 mm, vias 0 -> 2
- net SDIO_CMD: track 0.00 -> 50.8 mm, vias 0 -> 5
- net RX: track 0.00 -> 50.6 mm, vias 0 -> 2
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- added copper zone on B.Cu, net GND
- added copper zone on In1.Cu, net GND
- added copper zone on In2.Cu, net VCC_OBC
Other:
- board outline added: 90 x 90.2 mm
- copper layers 2 -> 4
- board text added: "GND"
- board text added: "NRST"
- board text added: "SWCLK"
- board text added: "SWDIO"
- board text added: "VCC"
