File: OBC/OBC_KICAD/microcontrolador.kicad_sch (KiCad schematic)
At the start: 21 parts, among them U2 STM32F405RGTx, Y1 ABMM-8.000MHZ-D-4-T

Commit message: Update
Parts:
- added C?: 10u, symbol Device:C
- added C?: 100n, symbol Device:C
- added CARD?: MICRO SD, MOLEX 5033981892:TF-SMD_503398-1892, symbol 503398-1892:503398-1892
- added R? (x5): 47K, symbol Device:R
- added R?: 100k, symbol Device:R
- renumbered C32 to C?, C29 to C?, C28 to C?, C26 to C?, C20 to C?, C25 to C?, C22 to C?, C23 to C?, C27 to C?, C21 to C?, C8 to C?, C6 to C?, C5 to C?, C7 to C?, C24 to C?, FB1 to FB?, R14 to R?, SwBoot1 to SwBoot?, SwReset1 to SwReset?, U2 to U?, Y1 to Y?
Connections:
- net +3.3VA: no longer C?.2, C?.2, FB?.2
- net +3V3: now also C?.2, C?.2, CARD?.4 (VDD), R?.1, R?.1, R?.1, R?.1, R?.1, R?.1
- net GND: now also C?.1, C?.1, CARD?.10, CARD?.11 (EH), CARD?.6 (VSS)
- net HSE_OUT: now also U?.6 (PH1)
- net MISO_BM: now reaches U?.10 (PC2)
- net MOSI_BM: now reaches U?.11 (PC3)
- net ELRS_UART_TX: now reaches U?.14 (PA0)
- net ELRS_UART_RX: now reaches U?.15 (PA1)
- net AP_CS_IMU: now reaches U?.20 (PA4)
- net CLK_IMU: now reaches U?.21 (PA5)
- net MISO_IMU: now reaches U?.22 (PA6)
- net MOSI_IMU: now reaches U?.23 (PA7)
- net CS_BM: now reaches U?.26 (PB0)
- net SCK_BM: now reaches U?.29 (PB10)
- net SDIO_D0: now reaches U?.39 (PC8)
- net SDIO_D0: now also CARD?.7 (DAT0), R?.2
- net SDIO_D1: now reaches U?.40 (PC9)
- net SDIO_D1: now also CARD?.8 (DAT1), R?.2
- net TX_VTX: now reaches U?.42 (PA9)
- net RX_VTX: now reaches U?.43 (PA10)
- net SDIO_D2: now reaches U?.51 (PC10)
- net SDIO_D2: now also CARD?.1 (DAT2), R?.2
- net SDIO_D3: now reaches U?.52 (PC11)
- net SDIO_D3: now also CARD?.2 (CD/DAT3), R?.2
- net SDIO_CLK: now reaches U?.53 (PC12)
- net SDIO_CLK: now also CARD?.5 (CLK)
- net SDIO_CMD: now reaches U?.54 (PD2)
- net SDIO_CMD: now also CARD?.3 (CMD), R?.2
- net SCL_MAG: now reaches U?.58 (PB6)
- net SDA_MAG: now reaches U?.59 (PB7)
- new net +3V3A: C?.2, C?.2, FB?.2
- new net CardDetect: CARD?.9, R?.2
Other:
- note added: "Esto es opcional, si se conecta al stm32 es una formaque te diga si hay una tarjeta insertada. pero no es necesario"
- note added: "MICRO SD"
- moved on the sheet: C?, FB?, R?, SwBoot?, SwReset?, Y?

Commit message: Agregar OCP TPS2052BDR y Watchdog STWD100
Agregue un OCP y un WatchDOg ,todo en la HOja con NOmbre Wtachdog.
Parts:
- gave numbers to parts that had none: 30
Connections:
- net +3V3: no longer C1.1, C2.1, C4.1, C6.1, C7.1, C9.1, U2.1 (VBAT), U2.19 (VDD), U2.32 (VDD), U2.48 (VDD), U2.64 (VDD)
- net EN1OBC: now reaches U2.24 (PC4)
- net PB1: now reaches U2.27 (PB1)
- net PB2: now reaches U2.28 (PB2)
- net NRST: now reaches U2.38 (PC7)
- net PB3: now reaches U2.55 (PB3)
- net WDI: now reaches U2.57 (PB5)
- net EN1P1: now reaches U2.8 (PC0)
- net EN2P2: now reaches U2.9 (PC1)
- new net VCC_OBC: C1.1, C2.1, C4.1, C6.1, C7.1, C9.1, U2.1 (VBAT), U2.19 (VDD), U2.32 (VDD), U2.48 (VDD), U2.64 (VDD)

Commit message: Cirtcuito Completo
Circuito Completo
Parts:
- removed C1: 4.7u, symbol Device:C_Polarized
- removed C11, C13: 16pF, symbol Device:C
- removed C14: 1u, symbol Device:C_Polarized
- removed Y1: ABMM-8.000MHZ-D-4-T, ABMM-8.000MHZ-D-4-T:ABMM25000MHZB2T, symbol ABMM-8_000MHZ-D-4-T:ABMM-8.000MHZ-D-4-T
- added C14: 1u, Capacitor_SMD:C_0805_2012Metric_Pad1.18x1.45mm_HandSolder, symbol Device:C
- added C18: 4.7u, Capacitor_SMD:C_0805_2012Metric_Pad1.18x1.45mm_HandSolder, symbol Device:C
- added C21, C22: 15pF, Capacitor_SMD:C_0805_2012Metric_Pad1.18x1.45mm_HandSolder, symbol Device:C
- added H1: MountingHole, MountingHole:MountingHole_3.2mm_M3_Pad_Via, symbol Mechanical:MountingHole
- added XTAL1: ECS-80-12-30BQ-JES-TR, esc_cristal:ECS-80-12_ECS, symbol ECS:ECS-80-12-30BQ-JES-TR
- C10, C12, C15, C16, C17, C2, C3, C4, C5, C6, C7, C8, C9: footprint (none) -> Capacitor_SMD:C_0805_2012Metric_Pad1.18x1.45mm_HandSolder
- CARD1: footprint MOLEX 5033981892:TF-SMD_503398-1892 -> Connector_Card:microSD_HC_Hirose_DM3AT-SF-PEJM5
- FB1: footprint (none) -> Inductor_SMD:L_Walsin_WLFM252009x
- R1, R2, R3, R4, R5, R6, R7: footprint (none) -> Resistor_SMD:R_0805_2012Metric_Pad1.20x1.40mm_HandSolder
- SwReset1: footprint (none) -> Button_Switch_SMD:SW_Push_1P1T_NO_CK_PTS125Sx43PSMTR
Connections:
- net +3.3VA is gone; now on net +3V3A: C12.1, U2.13 (VDDA)
- net +3V3 is gone; now on net VCC_OBC: C15.2, C16.2, CARD1.4 (VDD), FB1.1, R2.1, R3.1, R4.1, R5.1, R6.1, R7.1, SwBoot1.1 (C)
- net MISO_BM is gone; now on net CardDetect: U2.10 (PC2)
- net +3V3A: now also C14.1
- net GND: now also C14.2, C18.2, C21.2, C22.2, XTAL1.2, XTAL1.4
- net HSE_IN: now also C21.1, XTAL1.1
- net HSE_OUT: now also C22.1, XTAL1.3
- net VCC_OBC: now also C18.1
- net IEPS: now reaches U2.16 (PA2)
- net En_P2: now reaches U2.30 (PB11)
- net En_ADC: now reaches U2.33 (PB12)
- net En_COM: now reaches U2.34 (PB13)
- net AP_CS_IMU renamed CS
- net CLK_IMU renamed SCK
- net CS_BM: no longer names the net of U2.26 (PB0)
- net ELRS_UART_RX renamed RX
- net ELRS_UART_TX renamed TX
- net EN1OBC: no longer names the net of U2.24 (PC4)
- net EN1P1 renamed NRST_PROGRAM
- net EN2P2: no longer names the net of U2.9 (PC1)
- net LSE_IN: no longer names the net of U2.3 (PC14)
- net LSE_OUT: no longer names the net of U2.4 (PC15)
- net MISO_IMU renamed MISO
- net MOSI_BM: no longer names the net of U2.11 (PC3)
- net MOSI_IMU renamed MOSI
- net PB1: no longer names the net of U2.27 (PB1)
- net PB2: no longer names the net of U2.28 (PB2)
- net PB3: no longer names the net of U2.55 (PB3)
- net RX_VTX: no longer names the net of U2.43 (PA10)
- net SCK_BM renamed En_P1
- net SCL_MAG renamed SCL
- net SDA_MAG renamed SDA
- net TX_VTX: no longer names the net of U2.42 (PA9)
- no-connect marks 0 -> 22
Other:
- title: (none) -> David_Moises_Garcia_Sopino_Hoja1_IIS
- moved on the sheet: C17, R1, SwBoot1, SwReset1
