File: OBC/OBC_KICAD/untitled.kicad_sch (KiCad schematic)
At the start: 14 parts, among them J3 Conn_01x02, J4 Conn_01x02, U1 STWD100YNYWY3F, U3 TPS2052BDR, U4 TPS2052BDR

Commit message: Cirtcuito Completo
Circuito Completo
Parts:
- removed C18, C22: 22u, symbol Device:C
- removed C19, C21: 4.7u, symbol Device:C_Polarized
- removed J3, J4: Conn_01x02, Connector_JST:JST_PH_B2B-PH-K_1x02_P2.00mm_Vertical, symbol Connector_Generic:Conn_01x02
- removed R10, R9: 10k, symbol Device:R
- removed U3: TPS2052BDR, TPS2052BDR:SOIC127P599X175-8N, symbol TPS2052BDR:TPS2052BDR
- added C19: 4.7u, Capacitor_SMD:C_0805_2012Metric_Pad1.18x1.45mm_HandSolder, symbol Device:C
- added D2: 1N4148W, Diode_SMD:D_SOD-123, symbol Diode:1N4148W
- C20: footprint (none) -> Capacitor_SMD:C_0805_2012Metric_Pad1.18x1.45mm_HandSolder
- R12, R8: footprint (none) -> Resistor_SMD:R_0805_2012Metric_Pad1.20x1.40mm_HandSolder
Connections:
- net VCC_PL1 is gone; now on net GND: C20.2
- net +3V3: now also C19.1; no longer R12.1, U1.5 (VCC)
- net GND: now also C19.2; no longer C20.1
- net VCC_OBC: now also R12.1, U1.5 (VCC), D2.1 (K); no longer U4.7 (OUT1)
- net EN1OBC renamed Enable_EPStoOBC
- net PB3 renamed IEPS
- new net: C20.1, D2.2 (A), U4.7 (OUT1)
- no-connect marks 0 -> 4
Other:
- note removed: "OCP_Payloads"
- title: (none) -> David_Moises_Garcia_Sopino_Hoja3_IIS
- moved on the sheet: R8, U1
